File: PCB/MCU holder/mcu_holder.kicad_pcb (KiCad board)
At the start: 2 copper layers, 53.3 x 36.3 mm, 58 parts, among them J1 Conn_01x04_Female, J10 Conn_01x03_Female, J2 Conn_01x04_Female, J3 Conn_01x04_Female, J4 Conn_01x04_Female, J5 Conn_01x04_Female, J6 Conn_01x03_Female, J7 Conn_01x08_Female, J8 Conn_01x04_Female, J9 Conn_01x04_Female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

Commit message: fix mcu holder power circuit
Connections:
- SW17 pad 3: +5V -> Pogo_BAT+
- U1 pad 16: BAT+ -> Pogo_BAT+
Routing:
- net Pogo_BAT+: track 0.00 -> 41.2 mm
- net BAT+: track 43.9 -> 16.4 mm
- net +5V: track 62.3 -> 40.2 mm
