File: PCB/MCU holder/mcu_holder.kicad_sch (KiCad schematic)
At the start: 18 parts, among them J1 Conn_01x04_Female, J10 Conn_01x03_Female, J2 Conn_01x04_Female, J3 Conn_01x04_Female, J4 Conn_01x04_Female, J5 Conn_01x04_Female, J6 Conn_01x03_Female, J7 Conn_01x08_Female, J8 Conn_01x04_Female, J9 Conn_01x04_Female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

Commit message: fix mcu holder power circuit
Connections:
- net +5V: no longer SW17.3 (C)
- net BAT+: no longer U1.16 (BAT+)
- new net Pogo_BAT+: SW17.3 (C), U1.16 (BAT+)
